Commit message: added hand_yaw for arm

File: aero_shop/hand_yaw_s/urdf/hand_yaw.urdf.xacro (robot description, xacro)
@@ -43,5 +43,5 @@
     <origin xyz="0 0 0" rpy="0 0 0"/>
     <axis   xyz="0 0 1"/>
-    <limit lower="-2.0" upper="2.0" effort="100" velocity="2.0" />
+    <limit lower="0" upper="3.14" effort="100" velocity="2.0" />
     <dynamics damping="0.2" friction="0" />
   </joint>
