Commit message: fixed base_link in urdf

File: aero_shop/typeC_arm/urdf/aero_arm_typec.urdf.xacro (robot description, xacro)
@@ -10,16 +10,4 @@
   <xacro:macro name="aero_upper" params="base_link disable_mesh:=false r_hand_link:=r_hand_link">
   <link name="${base_link}">
-   <xacro:unless value="${disable_mesh}"><visual>
-     <origin xyz="0 0 0.01" rpy="0 0 0"/>
-     <geometry>
-       <mesh filename="package://aero_description/meshes/typeC_arm/WT_hip_base_F.DAE" scale="1 1 1"/>
-     </geometry>
-   </visual> </xacro:unless>
-   <xacro:unless value="${disable_mesh}"> <collision>
-      <origin xyz="0 0 0.01" rpy="0 0 0"/>
-      <geometry>
-        <mesh filename="package://aero_description/meshes/typeC_arm/WT_hip_base_F.DAE" scale="1 1 1"/>
-      </geometry>
-    </collision> </xacro:unless>
     <inertial>
       <origin xyz="0.0 0 0" rpy="0 0 0"/>

Commit message: tag

File: aero_shop/typeC_arm/urdf/aero_arm_typec.urdf.xacro (robot description, xacro)
@@ -131,5 +131,5 @@
     <child link="r_wrist_y_link"/>
     <dynamics damping="0.1"/>
-  <limit lower="-1.5707" upper="1.5707" effort="100" velocity="1.5" />
+  <limit lower="-2.0" upper="2.0" effort="100" velocity="1.5" />
   </joint>
   <joint name="r_wrist_p_joint" type="revolute">

Commit message: urdf fix

File: aero_shop/typeC_arm/urdf/aero_arm_typec.urdf.xacro (robot description, xacro)
@@ -105,5 +105,5 @@
     <child link="r_shoulder_link"/>
     <dynamics damping="0.1"/>
-  <limit lower="-1.57" upper="1.57" effort="3.14" velocity ="0.02"/>
+  <limit lower="-1.57" upper="1.57" effort="3.14" velocity ="0.6"/>
   </joint>
   <joint name="r_shoulder_p_joint" type="revolute">
@@ -126,5 +126,5 @@
   Please check aero_description/urdf/aero_arm_typec-->
   <joint name="r_wrist_y_joint" type="revolute">
-    <origin xyz="-0.035 0 0.0755" rpy="0 0 1.57"/>
+    <origin xyz="-0.035 0 0.0755" rpy="0 0 0"/>
 	  <axis xyz="0.0 0.0 1.0"/>
     <parent link="r_elbow_link"/>
@@ -134,5 +134,5 @@
   </joint>
   <joint name="r_wrist_p_joint" type="revolute">
-    <origin xyz="0 0 0.195" rpy="0 0 0"/>
+    <origin xyz="0 0 0.195" rpy="0 1.57 0"/>
 	  <axis xyz="0.0 1.0 0.0"/>
     <parent link="r_wrist_y_link"/>
@@ -142,5 +142,5 @@
   </joint>
   <joint name="r_wrist_r_joint" type="revolute">
-    <origin xyz="0 0 0" rpy="3.14 0 0"/>
+    <origin xyz="0 0 0" rpy="0 1.57 0"/>
 	  <axis xyz="1.0 0.0 0.0"/>
     <parent link="r_wrist_p_link"/>

Commit message: fixed

File: aero_shop/typeC_arm/urdf/aero_arm_typec.urdf.xacro (robot description, xacro)
@@ -131,5 +131,5 @@
     <child link="r_wrist_y_link"/>
     <dynamics damping="0.1"/>
-  <limit lower="-2.0" upper="2.0" effort="100" velocity="1.5" />
+  <limit lower="-3.14" upper="0.5" effort="100" velocity="1.5" />
   </joint>
   <joint name="r_wrist_p_joint" type="revolute">
@@ -147,5 +147,5 @@
     <child link="${r_hand_link}"/>
     <dynamics damping="0.1"/>
-    <limit lower="-0.698132" upper="1.57" effort="100" velocity="1.3" />
+    <limit lower="-0.6" upper="1.57" effort="100" velocity="1.3" />
   </joint>
   </xacro:macro>

Commit message: updated wrist_y limit

File: aero_shop/typeC_arm/urdf/aero_arm_typec.urdf.xacro (robot description, xacro)
@@ -131,5 +131,5 @@
     <child link="r_wrist_y_link"/>
     <dynamics damping="0.1"/>
-  <limit lower="-3.14" upper="0.5" effort="100" velocity="1.5" />
+  <limit lower="-3.3" upper="0.5" effort="100" velocity="1.5" />
   </joint>
   <joint name="r_wrist_p_joint" type="revolute">

Commit message: shop added

File: aero_shop/typeC_arm/urdf/aero_arm_typec.urdf.xacro (robot description, xacro)
@@ -134,18 +134,18 @@
   </joint>
   <joint name="r_wrist_p_joint" type="revolute">
-    <origin xyz="0 0 0.195" rpy="0 1.57 0"/>
-	  <axis xyz="0.0 1.0 0.0"/>
+    <origin xyz="0 0 0.195" rpy="0 0 0"/>
+	  <axis xyz="1.0 0.0 0.0"/>
     <parent link="r_wrist_y_link"/>
     <child link="r_wrist_p_link"/>
     <dynamics damping="0.1"/>
-  <limit lower="-0.15" upper="0.15" effort="100" velocity="1.3" />
+  <limit lower="-0.6" upper="1.57" effort="100" velocity="1.3" />
   </joint>
   <joint name="r_wrist_r_joint" type="revolute">
-    <origin xyz="0 0 0" rpy="0 1.57 0"/>
-	  <axis xyz="1.0 0.0 0.0"/>
+    <origin xyz="0 0 0" rpy="0 3.14 0"/>
+	  <axis xyz="0.0 1.0 0.0"/>
     <parent link="r_wrist_p_link"/>
     <child link="${r_hand_link}"/>
     <dynamics damping="0.1"/>
-    <limit lower="-0.6" upper="1.57" effort="100" velocity="1.3" />
+    <limit lower="-0.1" upper="0.1" effort="100" velocity="1.3" />
   </joint>
   </xacro:macro>
